File: PowerBricksBoard1.brd (EAGLE design)
At the start: 76.2 x 50.8 mm, 16 parts

Commit message: hi i updated it
Parts:
- moved R2 25.5 mm to (1.52, 25.8), flipped to the bottom, turned to 270 degrees
- moved R1 17.5 mm to (74.7, 16.8)
- moved D2 4.06 mm to (10.5, 49.3)
- moved D1 2.54 mm to (74.7, 34.9)
Routing:
- net 48V: track 31.5 -> 0.00 mm
- net N$2: track 1.45 -> 26.2 mm, vias 0 -> 1
- net 12V: track 17.4 -> 0.00 mm
- net N$1: track 1.45 -> 16.6 mm
- net ON/OFF: track 126.2 -> 127.2 mm, vias 0 -> 1
Changed lines of the file:
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@@
 <attribute name="VALUE" x="8.382" y="25.4" size="1.27" layer="27" rot="R90" align="center"/>
 </element>
-<element name="D1" library="SparkFun-LED" library_urn="urn:adsk.eagle:library:529" package="LED-0603" package3d_urn="urn:adsk.eagle:package:39354/1" value="" x="74.676" y="37.465" smashed="yes" rot="R90">
-<attribute name="NAME" x="74.041" y="37.465" size="0.6096" layer="25" font="vector" ratio="20" rot="R90" align="bottom-center"/>
-<attribute name="VALUE" x="75.311" y="37.465" size="0.6096" layer="27" font="vector" ratio="20" rot="R90" align="top-center"/>
-</element>
-<element name="D2" library="SparkFun-LED" library_urn="urn:adsk.eagle:library:529" package="LED-0603" package3d_urn="urn:adsk.eagle:package:39354/1" value="" x="14.605" y="49.276" smashed="yes">
-<attribute name="NAME" x="14.605" y="49.911" size="0.6096" layer="25" font="vector" ratio="20" align="bottom-center"/>
-<attribute name="VALUE" x="14.605" y="48.641" size="0.6096" layer="27" font="vector" ratio="20" align="top-center"/>
+<element name="D1" library="SparkFun-LED" library_urn="urn:adsk.eagle:library:529" package="LED-0603" package3d_urn="urn:adsk.eagle:package:39354/1" value="" x="74.676" y="34.925" smashed="yes" rot="R90">
+<attribute name="NAME" x="74.041" y="34.925" size="0.6096" layer="25" font="vector" ratio="20" rot="R90" align="bottom-center"/>
+<attribute name="VALUE" x="75.311" y="34.925" size="0.6096" layer="27" font="vector" ratio="20" rot="R90" align="top-center"/>
+</element>
+<element name="D2" library="SparkFun-LED" library_urn="urn:adsk.eagle:library:529" package="LED-0603" package3d_urn="urn:adsk.eagle:package:39354/1" value="" x="10.541" y="49.276" smashed="yes">
+<attribute name="NAME" x="10.541" y="49.911" size="0.6096" layer="25" font="vector" ratio="20" align="bottom-center"/>
+<attribute name="VALUE" x="10.541" y="48.641" size="0.6096" layer="27" font="vector" ratio="20" align="top-center"/>
 </element>
 <element name="H1" library="Mounting Holes" package="6-32-HOLE" package3d_urn="urn:adsk.eagle:package:24384748/2" value="6-32-HOLE" x="3.81" y="46.99" smashed="yes">
@@
 <attribute name="VALUE" x="72.39" y="1.524" size="0.6096" layer="27" font="vector" ratio="20" align="top-center"/>
 </element>
-<element name="R1" library="SparkFun-Resistors" library_urn="urn:adsk.eagle:library:532" package="0603" package3d_urn="urn:adsk.eagle:package:39650/1" value="470" x="74.676" y="34.29" smashed="yes" rot="R270">
-<attribute name="NAME" x="75.438" y="34.29" size="0.6096" layer="25" font="vector" ratio="20" rot="R270" align="bottom-center"/>
-<attribute name="PROD_ID" value=" " x="-16.764" y="-38.1" size="1.778" layer="27" rot="R270" display="off"/>
-<attribute name="VALUE" x="73.914" y="34.29" size="0.6096" layer="27" font="vector" ratio="20" rot="R270" align="top-center"/>
-</element>
-<element name="R2" library="SparkFun-Resistors" library_urn="urn:adsk.eagle:library:532" package="0603" package3d_urn="urn:adsk.eagle:package:39650/1" value="2400" x="11.43" y="49.276" smashed="yes" rot="R180">
-<attribute name="NAME" x="11.43" y="48.514" size="0.6096" layer="25" font="vector" ratio="20" rot="R180" align="bottom-center"/>
-<attribute name="PROD_ID" value=" " x="-64.77" y="140.716" size="1.778" layer="27" rot="R180" display="off"/>
-<attribute name="VALUE" x="11.43" y="50.038" size="0.6096" layer="27" font="vector" ratio="20" rot="R180" align="top-center"/>
+<element name="R1" library="SparkFun-Resistors" library_urn="urn:adsk.eagle:library:532" package="0603" package3d_urn="urn:adsk.eagle:package:39650/1" value="470" x="74.676" y="16.764" smashed="yes" rot="R270">
+<attribute name="NAME" x="75.438" y="16.764" size="0.6096" layer="25" font="vector" ratio="20" rot="R270" align="bottom-center"/>
+<attribute name="PROD_ID" value=" " x="-16.764" y="-55.626" size="1.778" layer="27" rot="R270" display="off"/>
+<attribute name="VALUE" x="73.914" y="16.764" size="0.6096" layer="27" font="vector" ratio="20" rot="R270" align="top-center"/>
+</element>
+<element name="R2" library="SparkFun-Resistors" library_urn="urn:adsk.eagle:library:532" package="0603" package3d_urn="urn:adsk.eagle:package:39650/1" value="2400" x="1.524" y="25.781" smashed="yes" rot="MR270">
+<attribute name="NAME" x="0.762" y="25.781" size="0.6096" layer="26" font="vector" ratio="20" rot="MR270" align="bottom-center"/>
+<attribute name="PROD_ID" value=" " x="92.964" y="-50.419" size="1.778" layer="28" rot="MR270" display="off"/>
+<attribute name="VALUE" x="2.286" y="25.781" size="0.6096" layer="28" font="vector" ratio="20" rot="MR270" align="top-center"/>
 </element>
 <element name="R3" library="SparkFun-Resistors" library_urn="urn:adsk.eagle:library:532" package="0603" package3d_urn="urn:adsk.eagle:package:39650/1" value=" " x="60.96" y="26.67" smashed="yes" rot="R270">
@@
 <contactref element="U$3" pad="1@10"/>
 <contactref element="U$2" pad="1"/>
-<wire x1="10.58" y1="49.276" x2="1.27" y2="39.966" width="0.254" layer="1"/>
-<wire x1="1.27" y1="39.966" x2="1.27" y2="21.59" width="0.254" layer="1"/>
 <polygon width="0.4064" layer="1" isolate="0.508" thermals="no">
 <vertex x="0.635" y="24.765"/>
@@
 <vertex x="2.032" y="39.624"/>
 </polygon>
-<wire x1="15.482" y1="49.276" x2="15.482" y2="47.232" width="0.254" layer="1"/>
+<wire x1="11.418" y1="49.276" x2="11.418" y2="47.232" width="0.254" layer="1"/>
 <via x="24.257" y="29.083" extent="1-16" drill="0.35"/>
 <via x="30.607" y="29.083" extent="1-16" drill="0.35"/>
@@
 <contactref element="U$2" pad="8"/>
 <contactref element="U$2" pad="9"/>
-<wire x1="74.676" y1="33.44" x2="74.93" y2="33.186" width="0.254" layer="1"/>
-<wire x1="74.93" y1="33.186" x2="74.93" y2="16.129" width="0.254" layer="1"/>
 <polygon width="0.4064" layer="16" isolate="0.508" thermals="no">
 <vertex x="25.908" y="15.494"/>
@@
 <via x="57.023" y="34.544" extent="1-16" drill="0.35"/>
 <via x="49.403" y="32.004" extent="1-16" drill="0.35"/>
-<wire x1="74.676" y1="38.342" x2="73.418" y2="38.342" width="0.254" layer="1"/>
+<wire x1="74.676" y1="35.802" x2="73.418" y2="35.802" width="0.254" layer="1"/>
 </signal>
 <signal name="ALERT">
@@
 <contactref element="R1" pad="1"/>
 <contactref element="D1" pad="A"/>
-<wire x1="74.676" y1="35.14" x2="74.676" y2="36.588" width="0.254" layer="1"/>
+<wire x1="74.93" y1="19.011" x2="74.676" y2="18.757" width="0.254" layer="1"/>
+<wire x1="74.676" y1="17.614" x2="74.676" y2="18.757" width="0.254" layer="1"/>
+<wire x1="74.93" y1="33.794" x2="74.676" y2="34.048" width="0.254" layer="1"/>
+<wire x1="74.93" y1="19.011" x2="74.93" y2="33.794" width="0.254" layer="1"/>
 </signal>
 <signal name="N$2">
 <contactref element="D2" pad="A"/>
 <contactref element="R2" pad="1"/>
-<wire x1="12.28" y1="49.276" x2="13.728" y2="49.276" width="0.254" layer="1"/>
+<wire x1="1.524" y1="26.631" x2="1.27" y2="26.885" width="0.254" layer="16"/>
+<via x="9.398" y="48.133" extent="1-16" drill="0.35"/>
+<wire x1="9.398" y1="48.133" x2="9.398" y2="49.01" width="0.254" layer="1"/>
+<wire x1="9.398" y1="49.01" x2="9.664" y2="49.276" width="0.254" layer="1"/>
+<wire x1="1.27" y1="26.885" x2="1.27" y2="40.005" width="0.254" layer="16"/>
+<wire x1="1.27" y1="40.005" x2="9.398" y2="48.133" width="0.254" layer="16"/>
 </signal>
 <signal name="DGND">
@@
 <contactref element="U$2" pad="2"/>
 <contactref element="U$3" pad="B"/>
-<wire x1="13.716" y1="25.4" x2="2.54" y2="25.4" width="0.4064" layer="16"/>
-<wire x1="2.54" y1="25.4" x2="1.27" y2="26.67" width="0.4064" layer="16"/>
-<wire x1="1.27" y1="26.67" x2="1.27" y2="40.0317125" width="0.4064" layer="16"/>
 <wire x1="74.93" y1="40.0317125" x2="74.93" y2="23.114" width="0.4064" layer="16"/>
 <wire x1="74.93" y1="23.114" x2="74.676" y2="22.86" width="0.4064" layer="16"/>
 <wire x1="74.676" y1="22.86" x2="73.66" y2="22.86" width="0.4064" layer="16"/>
-<wire x1="1.27" y1="40.0317125" x2="10.7682875" y2="49.53" width="0.4064" layer="16"/>
-<wire x1="10.7682875" y1="49.53" x2="65.4317125" y2="49.53" width="0.4064" layer="16"/>
-<wire x1="65.4317125" y1="49.53" x2="74.93" y2="40.0317125" width="0.4064" layer="16"/>
+<wire x1="13.716" y1="25.4" x2="2.794" y2="25.4" width="0.4064" layer="1"/>
+<wire x1="2.794" y1="25.4" x2="1.2192" y2="26.9748" width="0.4064" layer="1"/>
+<wire x1="1.2192" y1="26.9748" x2="1.2192" y2="39.9809125" width="0.4064" layer="1"/>
+<wire x1="7.62" y1="46.3817125" x2="7.62" y2="48.26" width="0.4064" layer="1"/>
+<via x="7.62" y="48.26" extent="1-16" drill="0.35"/>
+<wire x1="7.62" y1="48.26" x2="8.9408" y2="49.5808" width="0.4064" layer="16"/>
+<wire x1="8.9408" y1="49.5808" x2="65.3809125" y2="49.5808" width="0.4064" layer="16"/>
+<wire x1="1.2192" y1="39.9809125" x2="7.62" y2="46.3817125" width="0.4064" layer="1"/>
+<wire x1="65.3809125" y1="49.5808" x2="74.93" y2="40.0317125" width="0.4064" layer="16"/>
 </signal>
 </signals>

Commit message: Done but I still need to add a picture Owo
Parts:
- removed U$3: BRICK2DIST_C, Brick_Dist_Connector:BRICK2DIST_C
- added U$1: BRICK2DIST, Brick_Dist_Connector:BRICK2DIST_D2
- moved D1 43.9 mm to (33.2, 49.3), turned to 0 degrees
- moved R1 34.7 mm to (40.9, 24.9)
- moved D2 15.8 mm to (26.3, 49.3)
- moved R3 0.52 mm to (61.4, 26.3)
- moved R4 0.52 mm to (58.8, 26.3)
Connections:
- net 12V: now also U$1.2@1, U$1.2@10, U$1.2@11, U$1.2@12, U$1.2@13, U$1.2@14, U$1.2@15, U$1.2@16, U$1.2@17, U$1.2@18, U$1.2@19, U$1.2@2, U$1.2@20, U$1.2@3, U$1.2@4, U$1.2@5, U$1.2@6, U$1.2@7, U$1.2@8, U$1.2@9; no longer U$3.2@1, U$3.2@10, U$3.2@11, U$3.2@12, U$3.2@13, U$3.2@14, U$3.2@15, U$3.2@16, U$3.2@2, U$3.2@3, U$3.2@4, U$3.2@5, U$3.2@6, U$3.2@7, U$3.2@8, U$3.2@9
- net 12_GND: now also U$1.4@1, U$1.4@10, U$1.4@11, U$1.4@12, U$1.4@13, U$1.4@14, U$1.4@15, U$1.4@16, U$1.4@17, U$1.4@18, U$1.4@19, U$1.4@2, U$1.4@20, U$1.4@3, U$1.4@4, U$1.4@5, U$1.4@6, U$1.4@7, U$1.4@8, U$1.4@9; no longer U$3.4@1, U$3.4@10, U$3.4@11, U$3.4@12, U$3.4@13, U$3.4@14, U$3.4@15, U$3.4@16, U$3.4@2, U$3.4@3, U$3.4@4, U$3.4@5, U$3.4@6, U$3.4@7, U$3.4@8, U$3.4@9
- net 48V: now also U$1.1@1, U$1.1@10, U$1.1@2, U$1.1@3, U$1.1@4, U$1.1@5, U$1.1@6, U$1.1@7, U$1.1@8, U$1.1@9; no longer U$3.1@1, U$3.1@10, U$3.1@2, U$3.1@3, U$3.1@4, U$3.1@5, U$3.1@6, U$3.1@7, U$3.1@8, U$3.1@9
- net 48_GND: now also U$1.3@1, U$1.3@10, U$1.3@2, U$1.3@3, U$1.3@4, U$1.3@5, U$1.3@6, U$1.3@7, U$1.3@8, U$1.3@9; no longer U$3.3@1, U$3.3@10, U$3.3@2, U$3.3@3, U$3.3@4, U$3.3@5, U$3.3@6, U$3.3@7, U$3.3@8, U$3.3@9
- net ALERT: now also U$1.D; no longer U$3.D
- net C2: now also U$1.A; no longer U$3.A
- net CLK: now also U$1.C; no longer U$3.C
- net DATA: now also U$1.E; no longer U$3.E
- net ON/OFF: now also U$1.B; no longer U$3.B
Routing:
- net N$2: track 26.2 -> 41.4 mm
- net N$1: track 16.6 -> 27.1 mm
- net C2: track 14.2 -> 11.6 mm
- net ON/OFF: track 127.2 -> 125.3 mm
- net ALERT: track 7.66 -> 6.20 mm
- net CLK: track 7.43 -> 5.98 mm
- net 48_GND: track 2.04 -> 0.94 mm
- net DATA: track 7.88 -> 8.93 mm, vias 0 -> 1
- net N$3: track 7.93 -> 7.38 mm
- net 12_GND: track 1.26 -> 1.11 mm, vias 15 -> 13
Other:
- board text added: "12V"
- board text added: "48V"
- board text added: "ADDR1 = R3 Resistor ADDR0 = R4 Resistor Octal Address = 8*ADDR1 + ADDR0 0-12 and 40, 44, 45, and 55 address can’t be used (decimal)"
- board text added: "Octal digit -> Resistor(Kohm) _________ 0 | 10 1 | 15.4 2 | 23.7 3 | 36.5 4 | 54.9 5 | 84.5 6 | 130 7 | 200"
