File: PowerBricksBoard1.brd (EAGLE design)
At the start: 76.2 x 50.8 mm, 16 parts

Commit message: owo
Connections:
- net 48V renamed 48V_GND
- net N$3 renamed ADDR1
- net N$4 renamed ADDR0
- net N$5 renamed TRIM
Routing:
- net N$1: track 27.1 -> 31.0 mm
- net 12_GND: track 1.11 -> 2.38 mm
- net 48_GND: track 0.94 -> 1.63 mm
Other:
- board text added: "Trim up: 5.11 * 12 (100+ Delta )/(1.225* Delta) - 511/Delta - 10.2 = resistor to use in kOhm Where Delta is the % up for trim (10% = 10)"

Commit message: trim
Parts:
- R5: value 475k -> 510k
Changed lines of the file:
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@@
 <attribute name="VALUE" x="58.0644" y="26.3398" size="0.6096" layer="27" font="vector" ratio="20" rot="R270" align="top-center"/>
 </element>
-<element name="R5" library="SparkFun-Resistors" library_urn="urn:adsk.eagle:library:532" package="0603" package3d_urn="urn:adsk.eagle:package:39650/1" value="475k" x="60.96" y="22.733" smashed="yes" rot="R270">
+<element name="R5" library="SparkFun-Resistors" library_urn="urn:adsk.eagle:library:532" package="0603" package3d_urn="urn:adsk.eagle:package:39650/1" value="510k" x="60.96" y="22.733" smashed="yes" rot="R270">
 <attribute name="NAME" x="61.721996875" y="22.733003125" size="0.6096" layer="25" font="vector" ratio="20" rot="R270" align="bottom-center"/>
 <attribute name="PROD_ID" value=" " x="-30.479996875" y="-64.896996875" size="1.778" layer="27" rot="R270" display="off"/>

Commit message: Cleaning up git and exports for order
Parts:
- moved U$1 1.49 mm to (38.1, 25.4)
Routing:
- net ON/OFF: track 125.3 -> 126.9 mm
- net C2: track 11.6 -> 12.7 mm
- net ALERT: track 6.20 -> 5.14 mm
- net CLK: track 5.98 -> 4.92 mm
Changed lines of the file:
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@@
 <setting verticaltext="up"/>
 </settings>
-<grid distance="50" unitdist="mil" unit="mil" style="lines" multiple="1" display="no" altdistance="2" altunitdist="mil" altunit="mil"/>
+<grid distance="10" unitdist="mil" unit="mil" style="lines" multiple="1" display="no" altdistance="5" altunitdist="mil" altunit="mil"/>
 <layers>
 <layer number="1" name="Top" color="4" fill="1" visible="yes" active="yes"/>
@@
 </element>
 <element name="U$2" library="Delta Power Bricks - Q48SC12050NRDH" package="Q48SC12050NRDH" package3d_urn="urn:adsk.eagle:package:24241038/2" value="Q48SC12050NRDH" x="13.716" y="17.78" smashed="yes"/>
-<element name="U$1" library="Brick_Dist_Connector" package="BRICK2DIST_D2" value="BRICK2DIST" x="38.608" y="26.797" smashed="yes"/>
+<element name="U$1" library="Brick_Dist_Connector" package="BRICK2DIST_D2" value="BRICK2DIST" x="38.1" y="25.4" smashed="yes"/>
 </elements>
 <signals>
@@
 <vertex x="1.524" y="24.765"/>
 <vertex x="31.75" y="24.765"/>
-<vertex x="34.0868" y="22.4282"/>
-<vertex x="34.0868" y="14.1478"/>
+<vertex x="32.5628" y="23.9522"/>
+<vertex x="32.5628" y="12.6238"/>
 <vertex x="26.1366" y="6.1976"/>
 <vertex x="26.1366" y="3.5052"/>
@@
 <contactref element="U$2" pad="9"/>
 <polygon width="0.9144" layer="16" isolate="0.508">
-<vertex x="35.4076" y="13.6906"/>
+<vertex x="34.1376" y="12.4206"/>
 <vertex x="27.5336" y="5.8166"/>
 <vertex x="27.5336" y="-2.54"/>
@@
 <vertex x="67.31" y="19.05"/>
 <vertex x="61.722" y="24.638"/>
-<vertex x="38.5064" y="24.638"/>
-<vertex x="35.4076" y="21.5392"/>
+<vertex x="36.2204" y="24.638"/>
+<vertex x="34.1376" y="22.5552"/>
 </polygon>
 <polygon width="0.9144" layer="1" isolate="0.508">
@@
 <contactref element="U$2" pad="10"/>
 <contactref element="U$1" pad="A"/>
-<wire x1="74.168" y1="24.257" x2="73.5838" y2="24.257" width="0.254" layer="1"/>
-<wire x1="72.3646" y1="25.4762" x2="70.6628" y2="25.4762" width="0.254" layer="1"/>
-<wire x1="70.6628" y1="25.4762" x2="68.8086" y2="27.3304" width="0.254" layer="1"/>
-<wire x1="68.8086" y1="27.3304" x2="68.8086" y2="29.8704" width="0.254" layer="1"/>
+<wire x1="68.8086" y1="29.8704" x2="68.8086" y2="25.5524" width="0.254" layer="1"/>
 <wire x1="68.8086" y1="29.8704" x2="67.279" y2="31.4" width="0.254" layer="1"/>
 <wire x1="67.279" y1="31.4" x2="67.056" y2="31.4" width="0.254" layer="1"/>
-<wire x1="73.5838" y1="24.257" x2="72.3646" y2="25.4762" width="0.254" layer="1"/>
+<wire x1="72.39" y1="24.13" x2="73.66" y2="22.86" width="0.254" layer="1"/>
+<wire x1="68.8086" y1="25.5524" x2="70.231" y2="24.13" width="0.254" layer="1"/>
+<wire x1="70.231" y1="24.13" x2="72.39" y2="24.13" width="0.254" layer="1"/>
 </signal>
 <signal name="12_GND">
@@
 <vertex x="34.8742" y="27.9654"/>
 <vertex x="36.8046" y="26.035"/>
-<vertex x="55.118" y="26.035"/>
-<vertex x="57.658" y="28.575"/>
+<vertex x="60.706" y="26.035"/>
+<vertex x="63.246" y="28.575"/>
 <vertex x="67.564" y="28.575"/>
 <vertex x="73.66" y="34.671"/>
@@
 <wire x1="34.29" y1="48.26" x2="34.925" y2="47.625" width="0.1524" layer="1"/>
 <wire x1="34.925" y1="47.625" x2="35.306" y2="47.625" width="0.1524" layer="1"/>
+<wire x1="60.96" y1="39.37" x2="62.103" y2="39.624" width="0" layer="19" extent="1-1"/>
+<wire x1="50.673" y1="39.624" x2="50.8" y2="39.37" width="0" layer="19" extent="1-1"/>
 </signal>
 <signal name="ALERT">
 <contactref element="U$2" pad="13"/>
 <contactref element="U$1" pad="D"/>
-<wire x1="71.628" y1="29.337" x2="67.691" y2="25.4" width="0.254" layer="16"/>
-<wire x1="67.691" y1="25.4" x2="67.056" y2="25.4" width="0.254" layer="16"/>
+<wire x1="71.12" y1="27.94" x2="68.6562" y2="25.4" width="0.254" layer="16"/>
+<wire x1="68.6562" y1="25.4" x2="67.056" y2="25.4" width="0.254" layer="16"/>
 </signal>
 <signal name="DATA">
 <contactref element="U$2" pad="12"/>
 <contactref element="U$1" pad="E"/>
-<wire x1="67.056" y1="27.4" x2="68.5358" y2="28.8798" width="0.254" layer="16"/>
-<wire x1="69.9488" y1="28.8798" x2="68.5358" y2="28.8798" width="0.254" layer="16"/>
-<via x="69.9488" y="28.8798" extent="1-16" drill="0.35"/>
-<wire x1="69.9488" y1="28.8798" x2="70.8124" y2="28.0162" width="0.254" layer="1"/>
-<wire x1="70.8124" y1="28.0162" x2="73.3552" y2="28.0162" width="0.254" layer="1"/>
-<wire x1="73.3552" y1="28.0162" x2="74.168" y2="28.829" width="0.254" layer="1"/>
-<wire x1="74.168" y1="28.829" x2="74.168" y2="29.337" width="0.254" layer="1"/>
+<wire x1="67.056" y1="27.4" x2="68.469" y2="28.813" width="0.254" layer="16"/>
+<wire x1="68.469" y1="28.813" x2="68.5358" y2="28.8798" width="0.254" layer="16"/>
+<wire x1="68.5358" y1="28.8798" x2="70.136" y2="30.48" width="0.254" layer="16"/>
+<wire x1="70.136" y1="30.48" x2="71.628" y2="30.48" width="0.254" layer="16"/>
+<via x="71.628" y="30.48" extent="1-16" drill="0.35"/>
+<wire x1="71.628" y1="30.48" x2="73.66" y2="28.448" width="0.254" layer="1"/>
+<wire x1="73.66" y1="28.448" x2="73.66" y2="27.94" width="0.254" layer="1"/>
 </signal>
 <signal name="CLK">
 <contactref element="U$2" pad="14"/>
 <contactref element="U$1" pad="C"/>
-<wire x1="71.628" y1="26.797" x2="68.231" y2="23.4" width="0.254" layer="16"/>
-<wire x1="68.231" y1="23.4" x2="67.056" y2="23.4" width="0.254" layer="16"/>
+<wire x1="71.12" y1="25.4" x2="69.1962" y2="23.4" width="0.254" layer="16"/>
+<wire x1="69.1962" y1="23.4" x2="67.056" y2="23.4" width="0.254" layer="16"/>
 </signal>
 <signal name="N$1">
@@
 <wire x1="65.3809125" y1="49.5808" x2="74.62585625" y2="40.33585625" width="0.4064" layer="16"/>
 <contactref element="U$1" pad="B"/>
-<wire x1="74.62585625" y1="40.33585625" x2="74.62585625" y2="32.04195" width="0.4064" layer="16"/>
-<wire x1="72.9488" y1="25.5778" x2="71.628" y2="24.257" width="0.4064" layer="16"/>
-<wire x1="74.62585625" y1="32.04195" x2="72.9488" y2="30.36489375" width="0.4064" layer="16"/>
-<wire x1="72.9488" y1="30.36489375" x2="72.9488" y2="25.5778" width="0.4064" layer="16"/>
+<wire x1="74.62585625" y1="32.04195" x2="74.62585625" y2="40.33585625" width="0.4064" layer="16"/>
+<wire x1="71.12" y1="22.86" x2="72.39" y2="24.13" width="0.254" layer="16"/>
+<wire x1="72.39" y1="29.80609375" x2="74.62585625" y2="32.04195" width="0.254" layer="16"/>
+<wire x1="72.39" y1="24.13" x2="72.39" y2="29.80609375" width="0.254" layer="16"/>
 </signal>
 </signals>

Commit message: shrunk 0.025
Other:
- board size 76.2 x 50.8 mm -> 75.6 x 50.8 mm
- board text added: "=^..^="
- board text added: "~(^._.)"
Changed lines of the file:
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@@
 <board>
 <plain>
-<wire x1="0" y1="0" x2="76.2" y2="0" width="0" layer="20"/>
-<wire x1="76.2" y1="0" x2="76.2" y2="50.8" width="0" layer="20"/>
-<wire x1="76.2" y1="50.8" x2="0" y2="50.8" width="0" layer="20"/>
+<wire x1="0" y1="0" x2="75.565" y2="0" width="0" layer="20"/>
+<wire x1="75.565" y1="0" x2="75.565" y2="50.8" width="0" layer="20"/>
+<wire x1="75.565" y1="50.8" x2="0" y2="50.8" width="0" layer="20"/>
 <wire x1="0" y1="50.8" x2="0" y2="0" width="0" layer="20"/>
 <circle x="3.81" y="46.99" radius="3.048" width="0.1524" layer="25"/>
@@
 <text x="22.1996" y="48.5648" size="1.016" layer="25">48V</text>
 <text x="29.21" y="48.5902" size="1.016" layer="25">12V</text>
-<text x="35.56" y="2.54" size="1.016" layer="25">Trim up: 5.11 * 12 (100+ Delta )/(1.225* Delta)
+<text x="35.052" y="2.794" size="1.016" layer="25">Trim up: 5.11 * 12 (100+ Delta )/(1.225* Delta)
 - 511/Delta - 10.2 = resistor to use in kOhm
 Where Delta is the % up for trim (10% = 10) </text>
+<text x="22.86" y="35.56" size="1.778" layer="25">~(^._.)</text>
+<text x="22.606" y="13.716" size="1.778" layer="25">=^..^=</text>
 </plain>
 <attributes>
@@
 <vertex x="37.084" y="23.2664"/>
 </polygon>
-<via x="62.23" y="21.59" extent="1-16" drill="0.35"/>
-<via x="59.7154" y="24.257" extent="1-16" drill="0.35"/>
+<via x="62.484" y="21.082" extent="1-16" drill="0.35"/>
+<via x="62.3824" y="22.479" extent="1-16" drill="0.35"/>
 <via x="57.15" y="24.257" extent="1-16" drill="0.35"/>
 <via x="61.468" y="18.415" extent="1-16" drill="0.35"/>
@@
 <via x="49.53" y="22.987" extent="1-16" drill="0.35"/>
 <via x="57.531" y="20.066" extent="1-16" drill="0.35"/>
-<via x="42.2656" y="4.3942" extent="1-16" drill="0.35"/>
+<via x="40.9956" y="1.8542" extent="1-16" drill="0.35"/>
 <via x="42.9006" y="15.5448" extent="1-16" drill="0.35"/>
 <via x="32.4612" y="2.3114" extent="1-16" drill="0.35"/>
@@
 <via x="67.818" y="8.255" extent="1-16" drill="0.35"/>
 <via x="66.167" y="12.827" extent="1-16" drill="0.35"/>
-<via x="60.2742" y="6.8326" extent="1-16" drill="0.35"/>
+<via x="59.2582" y="1.7526" extent="1-16" drill="0.35"/>
 <via x="53.721" y="15.494" extent="1-16" drill="0.35"/>
-<via x="51.7652" y="4.5212" extent="1-16" drill="0.35"/>
+<via x="52.0192" y="1.7272" extent="1-16" drill="0.35"/>
 <contactref element="U$1" pad="2@20"/>
 <contactref element="U$1" pad="2@10"/>
@@
 <vertex x="68.58" y="31.75"/>
 <vertex x="70.739" y="31.75"/>
-<vertex x="73.66" y="34.671"/>
-<vertex x="73.66" y="40.005"/>
+<vertex x="73.279" y="34.29"/>
+<vertex x="73.279" y="40.386"/>
 <vertex x="65.024" y="48.641"/>
 </polygon>
@@
 <vertex x="63.246" y="28.575"/>
 <vertex x="67.564" y="28.575"/>
-<vertex x="73.66" y="34.671"/>
-<vertex x="73.66" y="44.323"/>
+<vertex x="73.533" y="34.544"/>
+<vertex x="73.533" y="44.45"/>
 <vertex x="65.405" y="52.578"/>
 <vertex x="35.814" y="52.578"/>
@@
 <via x="41.783" y="33.274" extent="1-16" drill="0.35"/>
 <via x="41.783" y="44.704" extent="1-16" drill="0.35"/>
-<via x="50.673" y="39.624" extent="1-16" drill="0.35"/>
-<via x="62.103" y="39.624" extent="1-16" drill="0.35"/>
+<via x="50.419" y="36.068" extent="1-16" drill="0.35"/>
+<via x="64.643" y="39.624" extent="1-16" drill="0.35"/>
 <via x="57.023" y="34.544" extent="1-16" drill="0.35"/>
 <via x="49.403" y="32.004" extent="1-16" drill="0.35"/>
@@
 <wire x1="34.29" y1="48.26" x2="34.925" y2="47.625" width="0.1524" layer="1"/>
 <wire x1="34.925" y1="47.625" x2="35.306" y2="47.625" width="0.1524" layer="1"/>
-<wire x1="60.96" y1="39.37" x2="62.103" y2="39.624" width="0" layer="19" extent="1-1"/>
-<wire x1="50.673" y1="39.624" x2="50.8" y2="39.37" width="0" layer="19" extent="1-1"/>
 </signal>
 <signal name="ALERT">
@@
 <wire x1="9.7028" y1="49.5808" x2="65.3809125" y2="49.5808" width="0.4064" layer="16"/>
 <wire x1="1.2192" y1="39.8285125" x2="9.271" y2="47.8803125" width="0.4064" layer="1"/>
-<wire x1="65.3809125" y1="49.5808" x2="74.62585625" y2="40.33585625" width="0.4064" layer="16"/>
+<wire x1="65.3809125" y1="49.5808" x2="74.24485625" y2="40.71685625" width="0.4064" layer="16"/>
 <contactref element="U$1" pad="B"/>
-<wire x1="74.62585625" y1="32.04195" x2="74.62585625" y2="40.33585625" width="0.4064" layer="16"/>
+<wire x1="74.24485625" y1="31.66095" x2="74.24485625" y2="40.71685625" width="0.4064" layer="16"/>
 <wire x1="71.12" y1="22.86" x2="72.39" y2="24.13" width="0.254" layer="16"/>
-<wire x1="72.39" y1="29.80609375" x2="74.62585625" y2="32.04195" width="0.254" layer="16"/>
+<wire x1="72.39" y1="29.80609375" x2="74.24485625" y2="31.66095" width="0.254" layer="16"/>
 <wire x1="72.39" y1="24.13" x2="72.39" y2="29.80609375" width="0.254" layer="16"/>
 </signal>

Commit message: 50mil smol
Parts:
- moved H2 1.27 mm to (71.1, 47.0)
- moved H4 1.27 mm to (71.1, 3.81)
- moved U$1 0.58 mm to (37.5, 25.4)
Routing:
- net ON/OFF: track 126.6 -> 125.6 mm
- net ALERT: track 5.14 -> 4.58 mm
- net CLK: track 4.92 -> 4.37 mm
Other:
- board size 75.6 x 50.8 mm -> 74.9 x 50.8 mm

Commit message: Revert "trim"
This reverts commit 0055e3f947d82e2e184832a38c8fbe8e78d74489.
Parts:
- R5: value 510k -> 475k
Changed lines of the file:
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@@
 <attribute name="VALUE" x="58.0644" y="26.3398" size="0.6096" layer="27" font="vector" ratio="20" rot="R270" align="top-center"/>
 </element>
-<element name="R5" library="SparkFun-Resistors" library_urn="urn:adsk.eagle:library:532" package="0603" package3d_urn="urn:adsk.eagle:package:39650/1" value="510k" x="60.96" y="22.733" smashed="yes" rot="R270">
+<element name="R5" library="SparkFun-Resistors" library_urn="urn:adsk.eagle:library:532" package="0603" package3d_urn="urn:adsk.eagle:package:39650/1" value="475k" x="60.96" y="22.733" smashed="yes" rot="R270">
 <attribute name="NAME" x="61.721996875" y="22.733003125" size="0.6096" layer="25" font="vector" ratio="20" rot="R270" align="bottom-center"/>
 <attribute name="PROD_ID" value=" " x="-30.479996875" y="-64.896996875" size="1.778" layer="27" rot="R270" display="off"/>

Commit message: Revert "Revert "trim""
This reverts commit 46b5d4a1c2a012013371b894087438f3b54206c6.
Parts:
- R5: value 475k -> 510k
Changed lines of the file:
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@@
 <attribute name="VALUE" x="58.0644" y="26.3398" size="0.6096" layer="27" font="vector" ratio="20" rot="R270" align="top-center"/>
 </element>
-<element name="R5" library="SparkFun-Resistors" library_urn="urn:adsk.eagle:library:532" package="0603" package3d_urn="urn:adsk.eagle:package:39650/1" value="475k" x="60.96" y="22.733" smashed="yes" rot="R270">
+<element name="R5" library="SparkFun-Resistors" library_urn="urn:adsk.eagle:library:532" package="0603" package3d_urn="urn:adsk.eagle:package:39650/1" value="510k" x="60.96" y="22.733" smashed="yes" rot="R270">
 <attribute name="NAME" x="61.721996875" y="22.733003125" size="0.6096" layer="25" font="vector" ratio="20" rot="R270" align="bottom-center"/>
 <attribute name="PROD_ID" value=" " x="-30.479996875" y="-64.896996875" size="1.778" layer="27" rot="R270" display="off"/>

Commit message: euhreiuhthjtrgrefwefrgyjgr
Connections:
- net 48V_GND renamed 48V
Changed lines of the file:
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@@
 </elements>
 <signals>
-<signal name="48V_GND">
-<contactref element="C1" pad="+"/>
-<contactref element="C2" pad="+"/>
-<contactref element="C4" pad="+"/>
-<contactref element="R2" pad="2"/>
-<contactref element="U$2" pad="1"/>
-<polygon width="0.9144" layer="1" isolate="0.508" rank="2">
-<vertex x="1.5494" y="24.765"/>
-<vertex x="34.4424" y="24.765"/>
-<vertex x="35.7632" y="23.4442"/>
-<vertex x="35.7632" y="15.8242"/>
-<vertex x="26.1366" y="6.1976"/>
-<vertex x="26.1366" y="3.6576"/>
-<vertex x="21.209" y="-1.27"/>
-<vertex x="11.43" y="-1.27"/>
-<vertex x="-1.27" y="11.43"/>
-<vertex x="-1.27" y="21.9456"/>
-</polygon>
-<polygon width="0.9144" layer="16" isolate="0.508" rank="2">
-<vertex x="1.524" y="24.765"/>
-<vertex x="31.75" y="24.765"/>
-<vertex x="32.5628" y="23.9522"/>
-<vertex x="32.5628" y="12.6238"/>
-<vertex x="26.1366" y="6.1976"/>
-<vertex x="26.1366" y="3.5052"/>
-<vertex x="21.3614" y="-1.27"/>
-<vertex x="11.43" y="-1.27"/>
-<vertex x="0" y="10.16"/>
-<vertex x="0" y="23.241"/>
-</polygon>
-<via x="17.78" y="22.86" extent="1-16" drill="0.35"/>
-<via x="25.4" y="22.86" extent="1-16" drill="0.35"/>
-<via x="29.21" y="22.86" extent="1-16" drill="0.35"/>
-<via x="25.0952" y="10.668" extent="1-16" drill="0.35"/>
-<via x="20.32" y="6.35" extent="1-16" drill="0.35"/>
-<via x="29.21" y="17.78" extent="1-16" drill="0.35"/>
-<via x="20.828" y="16.002" extent="1-16" drill="0.35"/>
-<via x="20.193" y="2.286" extent="1-16" drill="0.35"/>
-<via x="10.033" y="2.286" extent="1-16" drill="0.35"/>
-<via x="2.413" y="9.906" extent="1-16" drill="0.35"/>
-<via x="2.286" y="23.622" extent="1-16" drill="0.35"/>
-<via x="9.906" y="23.622" extent="1-16" drill="0.35"/>
-<via x="2.286" y="16.002" extent="1-16" drill="0.35"/>
-<via x="8.636" y="16.002" extent="1-16" drill="0.35"/>
-<contactref element="U$1" pad="1@1"/>
-<contactref element="U$1" pad="1@5"/>
-<contactref element="U$1" pad="1@6"/>
-<contactref element="U$1" pad="1@9"/>
-<contactref element="U$1" pad="1@10"/>
-<contactref element="U$1" pad="1@4"/>
-<contactref element="U$1" pad="1@3"/>
-<contactref element="U$1" pad="1@2"/>
-<contactref element="U$1" pad="1@8"/>
-<contactref element="U$1" pad="1@7"/>
-<polygon width="0.1524" layer="1" thermals="no">
-<vertex x="12.7508" y="20.32"/>
-<vertex x="14.5796" y="20.32"/>
-<vertex x="16.1036" y="18.796"/>
-<vertex x="16.1036" y="16.6878"/>
-<vertex x="14.859" y="15.4432"/>
-<vertex x="12.6492" y="15.4432"/>
-<vertex x="11.43" y="16.6624"/>
-<vertex x="11.43" y="18.9992"/>
-</polygon>
-<polygon width="0.1524" layer="16" thermals="no">
-<vertex x="12.7508" y="20.32"/>
-<vertex x="14.5796" y="20.32"/>
-<vertex x="16.1036" y="18.796"/>
-<vertex x="16.1036" y="16.6878"/>
-<vertex x="14.859" y="15.4432"/>
-<vertex x="12.6492" y="15.4432"/>
-<vertex x="11.43" y="16.6624"/>
-<vertex x="11.43" y="18.9992"/>
-</polygon>
-</signal>
 <signal name="48_GND">
 <contactref element="C1" pad="-"/>
@@
 <contactref element="U$2" pad="9"/>
 <polygon width="0.9144" layer="16" isolate="0.508">
-<vertex x="34.1376" y="12.4206"/>
+<vertex x="37.0586" y="15.3416"/>
 <vertex x="27.5336" y="5.8166"/>
 <vertex x="27.5336" y="-2.54"/>
@@
 <vertex x="67.31" y="19.05"/>
 <vertex x="61.722" y="24.638"/>
-<vertex x="36.2204" y="24.638"/>
-<vertex x="34.1376" y="22.5552"/>
+<vertex x="38.5064" y="24.638"/>
+<vertex x="37.0586" y="23.1902"/>
 </polygon>
 <polygon width="0.9144" layer="1" isolate="0.508">
@@
 <vertex x="31.4706" y="48.2346"/>
 <vertex x="31.4706" y="41.1734"/>
-<vertex x="34.8742" y="37.7698"/>
-<vertex x="34.8742" y="27.9654"/>
-<vertex x="36.8046" y="26.035"/>
+<vertex x="37.4142" y="35.2298"/>
+<vertex x="37.4142" y="27.4574"/>
+<vertex x="38.8366" y="26.035"/>
 <vertex x="60.706" y="26.035"/>
 <vertex x="63.246" y="28.575"/>
@@
 <wire x1="71.8058" y1="24.037071875" x2="71.8058" y2="29.22189375" width="0.4064" layer="16"/>
 </signal>
+<signal name="48V">
+<contactref element="U$2" pad="1"/>
+<contactref element="U$1" pad="1@1"/>
+<contactref element="U$1" pad="1@5"/>
+<contactref element="U$1" pad="1@6"/>
+<contactref element="U$1" pad="1@9"/>
+<contactref element="U$1" pad="1@10"/>
+<contactref element="U$1" pad="1@4"/>
+<contactref element="U$1" pad="1@3"/>
+<contactref element="U$1" pad="1@2"/>
+<contactref element="U$1" pad="1@8"/>
+<contactref element="U$1" pad="1@7"/>
+<contactref element="C1" pad="+"/>
+<contactref element="C2" pad="+"/>
+<contactref element="C4" pad="+"/>
+<contactref element="R2" pad="2"/>
+<polygon width="0.9144" layer="1" isolate="0.508" rank="2">
+<vertex x="1.5494" y="24.765"/>
+<vertex x="34.036" y="24.765"/>
+<vertex x="35.6108" y="23.1902"/>
+<vertex x="35.6108" y="15.6718"/>
+<vertex x="26.1366" y="6.1976"/>
+<vertex x="26.1366" y="3.6576"/>
+<vertex x="21.209" y="-1.27"/>
+<vertex x="11.43" y="-1.27"/>
+<vertex x="-1.27" y="11.43"/>
+<vertex x="-1.27" y="21.9456"/>
+</polygon>
+<polygon width="0.9144" layer="16" isolate="0.508" rank="2">
+<vertex x="1.524" y="24.765"/>
+<vertex x="34.036" y="24.765"/>
+<vertex x="35.6108" y="23.1902"/>
+<vertex x="35.6108" y="15.6718"/>
+<vertex x="26.1366" y="6.1976"/>
+<vertex x="26.1366" y="3.5052"/>
+<vertex x="21.3614" y="-1.27"/>
+<vertex x="11.43" y="-1.27"/>
+<vertex x="0" y="10.16"/>
+<vertex x="0" y="23.241"/>
+</polygon>
+<via x="17.78" y="22.86" extent="1-16" drill="0.35"/>
+<via x="25.4" y="22.86" extent="1-16" drill="0.35"/>
+<via x="29.21" y="22.86" extent="1-16" drill="0.35"/>
+<via x="25.0952" y="10.668" extent="1-16" drill="0.35"/>
+<via x="20.32" y="6.35" extent="1-16" drill="0.35"/>
+<via x="29.21" y="17.78" extent="1-16" drill="0.35"/>
+<via x="20.828" y="16.002" extent="1-16" drill="0.35"/>
+<via x="20.193" y="2.286" extent="1-16" drill="0.35"/>
+<via x="10.033" y="2.286" extent="1-16" drill="0.35"/>
+<via x="2.413" y="9.906" extent="1-16" drill="0.35"/>
+<via x="2.286" y="23.622" extent="1-16" drill="0.35"/>
+<via x="9.906" y="23.622" extent="1-16" drill="0.35"/>
+<via x="2.286" y="16.002" extent="1-16" drill="0.35"/>
+<via x="8.636" y="16.002" extent="1-16" drill="0.35"/>
+<polygon width="0.1524" layer="1" thermals="no">
+<vertex x="12.7508" y="20.32"/>
+<vertex x="14.5796" y="20.32"/>
+<vertex x="16.1036" y="18.796"/>
+<vertex x="16.1036" y="16.6878"/>
+<vertex x="14.859" y="15.4432"/>
+<vertex x="12.6492" y="15.4432"/>
+<vertex x="11.43" y="16.6624"/>
+<vertex x="11.43" y="18.9992"/>
+</polygon>
+<polygon width="0.1524" layer="16" thermals="no">
+<vertex x="12.7508" y="20.32"/>
+<vertex x="14.5796" y="20.32"/>
+<vertex x="16.1036" y="18.796"/>
+<vertex x="16.1036" y="16.6878"/>
+<vertex x="14.859" y="15.4432"/>
+<vertex x="12.6492" y="15.4432"/>
+<vertex x="11.43" y="16.6624"/>
+<vertex x="11.43" y="18.9992"/>
+</polygon>
+</signal>
 </signals>
