File: PowerBricksBoard1.sch (EAGLE design)
At the start: 15 parts

Commit message: layout
Parts:
- removed U$2: PMBUSTABLE, PMBUS Resistors:PMBUSTABLE
- added R3: (no value), SparkFun-Resistors:RESISTOR0603
Connections:
- net DGND: now also R3.1; no longer U$2.1
- net N$3: now also R3.2; no longer U$2.2
Changed lines of the file:
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@@
 <part name="C3" library="UCM1H331MNL1GS" deviceset="UCM1H331MNL1GS" device=""/>
 <part name="R4" library="SparkFun-Resistors" library_urn="urn:adsk.eagle:library:532" deviceset="RESISTOR" device="0603" package3d_urn="urn:adsk.eagle:package:39650/1" value=" "/>
-<part name="U$2" library="PMBUS Resistors" deviceset="PMBUSTABLE" device=""/>
+<part name="R3" library="SparkFun-Resistors" library_urn="urn:adsk.eagle:library:532" deviceset="RESISTOR" device="0603" package3d_urn="urn:adsk.eagle:package:39650/1" value=" "/>
 </parts>
 <sheets>
@@
 <attribute name="VALUE" x="-33.02" y="18.796" size="1.778" layer="96" font="vector" align="top-center"/>
 </instance>
-<instance part="U$2" gate="G$1" x="-33.02" y="27.94" smashed="yes">
+<instance part="R3" gate="G$1" x="-33.02" y="27.94" smashed="yes">
 <attribute name="NAME" x="-33.02" y="29.464" size="1.778" layer="95" font="vector" align="bottom-center"/>
+<attribute name="VALUE" x="-33.02" y="26.416" size="1.778" layer="96" font="vector" align="top-center"/>
 </instance>
 </instances>
@@
 <pinref part="R4" gate="G$1" pin="1"/>
 <wire x1="-45.72" y1="27.94" x2="-38.1" y2="27.94" width="0.1524" layer="91"/>
-<pinref part="U$2" gate="G$1" pin="1"/>
+<pinref part="R3" gate="G$1" pin="1"/>
 </segment>
 </net>
@@
 <pinref part="U$1" gate="G$1" pin="ADDR1"/>
 <wire x1="-27.94" y1="27.94" x2="-17.78" y2="27.94" width="0.1524" layer="91"/>
-<pinref part="U$2" gate="G$1" pin="2"/>
+<pinref part="R3" gate="G$1" pin="2"/>
 </segment>
 </net>
@@
 </drawing>
 <compatibility>
-<note version="6.3" minversion="6.2.2" severity="warning">
-Since Version 6.2.2 text objects can contain more than one line,
-which will not be processed correctly with this version.
-</note>
 <note version="8.2" severity="warning">
 Since Version 8.2, EAGLE supports online libraries. The ids

Commit message: owo
Connections:
- net 12V: now also U$1.SENSE(+)
- net 12_GND: now also U$1.SENSE(-)
- net ON/OFF: now also U$1.C2
Changed lines of the file:
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@@
 <net name="12V" class="0">
 <segment>
-<wire x1="17.78" y1="20.32" x2="33.02" y2="20.32" width="0.1524" layer="91"/>
+<wire x1="17.78" y1="20.32" x2="25.4" y2="20.32" width="0.1524" layer="91"/>
 <label x="33.02" y="20.32" size="1.778" layer="95" xref="yes"/>
 <pinref part="U$1" gate="G$1" pin="VOUT(+)"/>
+<pinref part="U$1" gate="G$1" pin="SENSE(+)"/>
+<wire x1="25.4" y1="20.32" x2="33.02" y2="20.32" width="0.1524" layer="91"/>
+<wire x1="17.78" y1="12.7" x2="25.4" y2="12.7" width="0.1524" layer="91"/>
+<wire x1="25.4" y1="12.7" x2="25.4" y2="20.32" width="0.1524" layer="91"/>
+<junction x="25.4" y="20.32"/>
 </segment>
 <segment>
@@
 <pinref part="U$1" gate="G$1" pin="ON/OFF"/>
 </segment>
+<segment>
+<wire x1="17.78" y1="27.94" x2="30.48" y2="27.94" width="0.1524" layer="91"/>
+<label x="30.48" y="27.94" size="1.778" layer="95" xref="yes"/>
+<pinref part="U$1" gate="G$1" pin="C2"/>
+</segment>
 </net>
 <net name="12_GND" class="0">
 <segment>
-<wire x1="17.78" y1="-10.16" x2="33.02" y2="-10.16" width="0.1524" layer="91"/>
+<wire x1="17.78" y1="-10.16" x2="25.4" y2="-10.16" width="0.1524" layer="91"/>
 <label x="33.02" y="-10.16" size="1.778" layer="95" xref="yes"/>
 <pinref part="U$1" gate="G$1" pin="VOUT(-)"/>
+<pinref part="U$1" gate="G$1" pin="SENSE(-)"/>
+<wire x1="25.4" y1="-10.16" x2="33.02" y2="-10.16" width="0.1524" layer="91"/>
+<wire x1="17.78" y1="-2.54" x2="25.4" y2="-2.54" width="0.1524" layer="91"/>
+<wire x1="25.4" y1="-2.54" x2="25.4" y2="-10.16" width="0.1524" layer="91"/>
+<junction x="25.4" y="-10.16"/>
 </segment>
 <segment>

Commit message: schematic, resistor calcs, routing
Parts:
- added R5: 475k, SparkFun-Resistors:RESISTOR0603
- R2: value 470 -> 2400
Connections:
- new net N$5: R5.1, U$1.TRIM
- net 12V: now also R5.2
Other:
- moved on the sheet: D1, D2, R1, R2
Changed lines of the file:
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@@
 <part name="R1" library="SparkFun-Resistors" library_urn="urn:adsk.eagle:library:532" deviceset="RESISTOR" device="0603" package3d_urn="urn:adsk.eagle:package:39650/1" value="470"/>
 <part name="D2" library="SparkFun-LED" library_urn="urn:adsk.eagle:library:529" deviceset="LED" device="0603" package3d_urn="urn:adsk.eagle:package:39354/1"/>
-<part name="R2" library="SparkFun-Resistors" library_urn="urn:adsk.eagle:library:532" deviceset="RESISTOR" device="0603" package3d_urn="urn:adsk.eagle:package:39650/1" value="470"/>
 <part name="U$6" library="Dist_to_Brickboard_Connector_brick" deviceset="BRICKBOARD_TSW_14X2" device="" package3d_urn="urn:adsk.eagle:package:23225958/2"/>
 <part name="C1" library="UCM1H331MNL1GS" deviceset="UCM1H331MNL1GS" device=""/>
@@
 <part name="R4" library="SparkFun-Resistors" library_urn="urn:adsk.eagle:library:532" deviceset="RESISTOR" device="0603" package3d_urn="urn:adsk.eagle:package:39650/1" value=" "/>
 <part name="R3" library="SparkFun-Resistors" library_urn="urn:adsk.eagle:library:532" deviceset="RESISTOR" device="0603" package3d_urn="urn:adsk.eagle:package:39650/1" value=" "/>
+<part name="R2" library="SparkFun-Resistors" library_urn="urn:adsk.eagle:library:532" deviceset="RESISTOR" device="0603" package3d_urn="urn:adsk.eagle:package:39650/1" value="2400"/>
+<part name="R5" library="SparkFun-Resistors" library_urn="urn:adsk.eagle:library:532" deviceset="RESISTOR" device="0603" package3d_urn="urn:adsk.eagle:package:39650/1" value="475k"/>
 </parts>
 <sheets>
@@
 <instance part="H4" gate="G$1" x="109.22" y="10.16" smashed="yes"/>
 <instance part="U$1" gate="G$1" x="0" y="0" smashed="yes"/>
-<instance part="D1" gate="G$1" x="-93.98" y="-15.24" smashed="yes">
-<attribute name="NAME" x="-97.409" y="-19.812" size="1.778" layer="95" font="vector" rot="R90"/>
-<attribute name="VALUE" x="-92.075" y="-19.812" size="1.778" layer="96" font="vector" rot="R90" align="top-left"/>
-</instance>
-<instance part="R1" gate="G$1" x="-93.98" y="-5.08" smashed="yes" rot="R90">
-<attribute name="NAME" x="-95.504" y="-5.08" size="1.778" layer="95" font="vector" rot="R90" align="bottom-center"/>
-<attribute name="VALUE" x="-92.456" y="-5.08" size="1.778" layer="96" font="vector" rot="R90" align="top-center"/>
-</instance>
-<instance part="D2" gate="G$1" x="-66.04" y="-15.24" smashed="yes">
-<attribute name="NAME" x="-69.469" y="-19.812" size="1.778" layer="95" font="vector" rot="R90"/>
-<attribute name="VALUE" x="-64.135" y="-19.812" size="1.778" layer="96" font="vector" rot="R90" align="top-left"/>
-</instance>
-<instance part="R2" gate="G$1" x="-66.04" y="-5.08" smashed="yes" rot="R90">
-<attribute name="NAME" x="-67.564" y="-5.08" size="1.778" layer="95" font="vector" rot="R90" align="bottom-center"/>
-<attribute name="VALUE" x="-64.516" y="-5.08" size="1.778" layer="96" font="vector" rot="R90" align="top-center"/>
+<instance part="D1" gate="G$1" x="-101.6" y="-38.1" smashed="yes">
+<attribute name="NAME" x="-105.029" y="-42.672" size="1.778" layer="95" font="vector" rot="R90"/>
+<attribute name="VALUE" x="-99.695" y="-42.672" size="1.778" layer="96" font="vector" rot="R90" align="top-left"/>
+</instance>
+<instance part="R1" gate="G$1" x="-101.6" y="-22.86" smashed="yes" rot="R90">
+<attribute name="NAME" x="-103.124" y="-22.86" size="1.778" layer="95" font="vector" rot="R90" align="bottom-center"/>
+<attribute name="VALUE" x="-100.076" y="-22.86" size="1.778" layer="96" font="vector" rot="R90" align="top-center"/>
+</instance>
+<instance part="D2" gate="G$1" x="-73.66" y="-38.1" smashed="yes">
+<attribute name="NAME" x="-77.089" y="-42.672" size="1.778" layer="95" font="vector" rot="R90"/>
+<attribute name="VALUE" x="-71.755" y="-42.672" size="1.778" layer="96" font="vector" rot="R90" align="top-left"/>
 </instance>
 <instance part="U$6" gate="G$1" x="35.56" y="66.04" smashed="yes">
@@
 <attribute name="NAME" x="-33.02" y="29.464" size="1.778" layer="95" font="vector" align="bottom-center"/>
 <attribute name="VALUE" x="-33.02" y="26.416" size="1.778" layer="96" font="vector" align="top-center"/>
+</instance>
+<instance part="R2" gate="G$1" x="-73.66" y="-22.86" smashed="yes" rot="R90">
+<attribute name="NAME" x="-75.184" y="-22.86" size="1.778" layer="95" font="vector" rot="R90" align="bottom-center"/>
+<attribute name="VALUE" x="-72.136" y="-22.86" size="1.778" layer="96" font="vector" rot="R90" align="top-center"/>
+</instance>
+<instance part="R5" gate="G$1" x="35.56" y="5.08" smashed="yes">
+<attribute name="NAME" x="35.56" y="6.604" size="1.778" layer="95" font="vector" align="bottom-center"/>
+<attribute name="VALUE" x="35.56" y="3.556" size="1.778" layer="96" font="vector" align="top-center"/>
 </instance>
 </instances>
@@
 </segment>
 <segment>
+<wire x1="-73.66" y1="-17.78" x2="-73.66" y2="-12.7" width="0.1524" layer="91"/>
+<label x="-73.66" y="-12.7" size="1.778" layer="95" rot="R90" xref="yes"/>
 <pinref part="R2" gate="G$1" pin="2"/>
-<wire x1="-66.04" y1="0" x2="-66.04" y2="5.08" width="0.1524" layer="91"/>
-<label x="-66.04" y="5.08" size="1.778" layer="95" rot="R90" xref="yes"/>
 </segment>
 </net>
@@
 <segment>
 <pinref part="D2" gate="G$1" pin="C"/>
-<wire x1="-66.04" y1="-20.32" x2="-66.04" y2="-27.94" width="0.1524" layer="91"/>
-<label x="-66.04" y="-27.94" size="1.778" layer="95" rot="R270" xref="yes"/>
+<wire x1="-73.66" y1="-43.18" x2="-73.66" y2="-50.8" width="0.1524" layer="91"/>
+<label x="-73.66" y="-50.8" size="1.778" layer="95" rot="R270" xref="yes"/>
 </segment>
 </net>
@@
 <segment>
 <wire x1="17.78" y1="20.32" x2="25.4" y2="20.32" width="0.1524" layer="91"/>
-<label x="33.02" y="20.32" size="1.778" layer="95" xref="yes"/>
+<label x="55.88" y="20.32" size="1.778" layer="95" xref="yes"/>
 <pinref part="U$1" gate="G$1" pin="VOUT(+)"/>
 <pinref part="U$1" gate="G$1" pin="SENSE(+)"/>
-<wire x1="25.4" y1="20.32" x2="33.02" y2="20.32" width="0.1524" layer="91"/>
+<wire x1="25.4" y1="20.32" x2="50.8" y2="20.32" width="0.1524" layer="91"/>
+<wire x1="50.8" y1="20.32" x2="55.88" y2="20.32" width="0.1524" layer="91"/>
 <wire x1="17.78" y1="12.7" x2="25.4" y2="12.7" width="0.1524" layer="91"/>
 <wire x1="25.4" y1="12.7" x2="25.4" y2="20.32" width="0.1524" layer="91"/>
 <junction x="25.4" y="20.32"/>
+<wire x1="50.8" y1="5.08" x2="50.8" y2="20.32" width="0.1524" layer="91"/>
+<junction x="50.8" y="20.32"/>
+<pinref part="R5" gate="G$1" pin="2"/>
+<wire x1="40.64" y1="5.08" x2="50.8" y2="5.08" width="0.1524" layer="91"/>
 </segment>
 <segment>
 <pinref part="R1" gate="G$1" pin="2"/>
-<wire x1="-93.98" y1="0" x2="-93.98" y2="5.08" width="0.1524" layer="91"/>
-<label x="-93.98" y="5.08" size="1.778" layer="95" rot="R90" xref="yes"/>
+<wire x1="-101.6" y1="-17.78" x2="-101.6" y2="-12.7" width="0.1524" layer="91"/>
+<label x="-101.6" y="-12.7" size="1.778" layer="95" rot="R90" xref="yes"/>
 </segment>
 <segment>
@@
 <segment>
 <pinref part="D1" gate="G$1" pin="C"/>
-<wire x1="-93.98" y1="-20.32" x2="-93.98" y2="-27.94" width="0.1524" layer="91"/>
-<label x="-93.98" y="-27.94" size="1.778" layer="95" rot="R270" xref="yes"/>
+<wire x1="-101.6" y1="-43.18" x2="-101.6" y2="-50.8" width="0.1524" layer="91"/>
+<label x="-101.6" y="-50.8" size="1.778" layer="95" rot="R270" xref="yes"/>
 </segment>
 <segment>
@@
 <pinref part="R1" gate="G$1" pin="1"/>
 <pinref part="D1" gate="G$1" pin="A"/>
-<wire x1="-93.98" y1="-10.16" x2="-93.98" y2="-12.7" width="0.1524" layer="91"/>
+<wire x1="-101.6" y1="-27.94" x2="-101.6" y2="-35.56" width="0.1524" layer="91"/>
 </segment>
 </net>
 <net name="N$2" class="0">
 <segment>
+<pinref part="D2" gate="G$1" pin="A"/>
 <pinref part="R2" gate="G$1" pin="1"/>
-<pinref part="D2" gate="G$1" pin="A"/>
-<wire x1="-66.04" y1="-10.16" x2="-66.04" y2="-12.7" width="0.1524" layer="91"/>
+<wire x1="-73.66" y1="-35.56" x2="-73.66" y2="-27.94" width="0.1524" layer="91"/>
 </segment>
 </net>
@@
 </segment>
 </net>
+<net name="N$5" class="0">
+<segment>
+<pinref part="U$1" gate="G$1" pin="TRIM"/>
+<wire x1="30.48" y1="5.08" x2="17.78" y2="5.08" width="0.1524" layer="91"/>
+<pinref part="R5" gate="G$1" pin="1"/>
+</segment>
+</net>

Commit message: yes these changes are very pog
Other:
- note added: "ADDR1 = R3 Resistor ADDR0 = R4 Resistor Octal Address = 8*ADDR1 + ADDR0"
- note added: "Octal digit -> Resistor(Kohm) _________ 0 | 10 1 | 15.4 2 | 23.7 3 | 36.5 4 | 54.9 5 | 84.5 6 | 130 7 | 200"
Changed lines of the file:
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@@
 <sheet>
 <plain>
+<text x="81.28" y="-30.48" size="1.778" layer="91">Octal digit -&gt; Resistor(Kohm)
+_________
+ 0  |  10
+ 1  |  15.4
+ 2  |  23.7
+ 3  |  36.5
+ 4  |  54.9
+ 5  |  84.5
+ 6  |  130
+ 7  |  200</text>
+<text x="81.28" y="-43.18" size="1.778" layer="91">ADDR1 = R3 Resistor
+ADDR0 = R4 Resistor
+Octal Address = 8*ADDR1 + ADDR0 </text>
 </plain>
 <instances>
@@
 </drawing>
 <compatibility>
+<note version="6.3" minversion="6.2.2" severity="warning">
+Since Version 6.2.2 text objects can contain more than one line,
+which will not be processed correctly with this version.
+</note>
 <note version="8.2" severity="warning">
 Since Version 8.2, EAGLE supports online libraries. The ids

Commit message: brick update
Parts:
- H1, H2, H3, H4: value STAND-OFF -> 6-32-HOLE; device SparkFun-Hardware:STAND-OFF -> Mounting Holes:6-32-HOLE
Changed lines of the file:
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@@
 <parts>
 <part name="FRAME1" library="frames" library_urn="urn:adsk.eagle:library:229" deviceset="A4L-LOC" device=""/>
-<part name="H1" library="SparkFun-Hardware" library_urn="urn:adsk.eagle:library:519" deviceset="STAND-OFF" device="" package3d_urn="urn:adsk.eagle:package:38630/1"/>
-<part name="H2" library="SparkFun-Hardware" library_urn="urn:adsk.eagle:library:519" deviceset="STAND-OFF" device="" package3d_urn="urn:adsk.eagle:package:38630/1"/>
-<part name="H3" library="SparkFun-Hardware" library_urn="urn:adsk.eagle:library:519" deviceset="STAND-OFF" device="" package3d_urn="urn:adsk.eagle:package:38630/1"/>
-<part name="H4" library="SparkFun-Hardware" library_urn="urn:adsk.eagle:library:519" deviceset="STAND-OFF" device="" package3d_urn="urn:adsk.eagle:package:38630/1"/>
 <part name="U$1" library="Q48SC12050NRDH" deviceset="Q48SC12050NRDH" device=""/>
 <part name="D1" library="SparkFun-LED" library_urn="urn:adsk.eagle:library:529" deviceset="LED" device="0603" package3d_urn="urn:adsk.eagle:package:39354/1"/>
@@
 <part name="R2" library="SparkFun-Resistors" library_urn="urn:adsk.eagle:library:532" deviceset="RESISTOR" device="0603" package3d_urn="urn:adsk.eagle:package:39650/1" value="2400"/>
 <part name="R5" library="SparkFun-Resistors" library_urn="urn:adsk.eagle:library:532" deviceset="RESISTOR" device="0603" package3d_urn="urn:adsk.eagle:package:39650/1" value="475k"/>
+<part name="H1" library="Mounting Holes" deviceset="6-32-HOLE" device="" package3d_urn="urn:adsk.eagle:package:24384748/2"/>
+<part name="H2" library="Mounting Holes" deviceset="6-32-HOLE" device="" package3d_urn="urn:adsk.eagle:package:24384748/2"/>
+<part name="H3" library="Mounting Holes" deviceset="6-32-HOLE" device="" package3d_urn="urn:adsk.eagle:package:24384748/2"/>
+<part name="H4" library="Mounting Holes" deviceset="6-32-HOLE" device="" package3d_urn="urn:adsk.eagle:package:24384748/2"/>
 </parts>
 <sheets>
@@
 <attribute name="SHEET" x="100.965" y="-73.66" size="2.54" layer="94"/>
 </instance>
-<instance part="H1" gate="G$1" x="109.22" y="15.24" smashed="yes"/>
-<instance part="H2" gate="G$1" x="104.14" y="15.24" smashed="yes"/>
-<instance part="H3" gate="G$1" x="104.14" y="10.16" smashed="yes"/>
-<instance part="H4" gate="G$1" x="109.22" y="10.16" smashed="yes"/>
 <instance part="U$1" gate="G$1" x="0" y="0" smashed="yes"/>
 <instance part="D1" gate="G$1" x="-101.6" y="-38.1" smashed="yes">
@@
 <attribute name="VALUE" x="35.56" y="3.556" size="1.778" layer="96" font="vector" align="top-center"/>
 </instance>
+<instance part="H1" gate="G$1" x="96.52" y="25.4" smashed="yes">
+<attribute name="NAME" x="96.52" y="27.94" size="1.016" layer="95" align="bottom-center"/>
+<attribute name="VALUE" x="96.52" y="22.86" size="1.016" layer="95" align="top-center"/>
+</instance>
+<instance part="H2" gate="G$1" x="101.6" y="25.4" smashed="yes">
+<attribute name="NAME" x="101.6" y="27.94" size="1.016" layer="95" align="bottom-center"/>
+<attribute name="VALUE" x="101.6" y="22.86" size="1.016" layer="95" align="top-center"/>
+</instance>
+<instance part="H3" gate="G$1" x="106.68" y="25.4" smashed="yes">
+<attribute name="NAME" x="106.68" y="27.94" size="1.016" layer="95" align="bottom-center"/>
+<attribute name="VALUE" x="106.68" y="22.86" size="1.016" layer="95" align="top-center"/>
+</instance>
+<instance part="H4" gate="G$1" x="111.76" y="25.4" smashed="yes">
+<attribute name="NAME" x="111.76" y="27.94" size="1.016" layer="95" align="bottom-center"/>
+<attribute name="VALUE" x="111.76" y="22.86" size="1.016" layer="95" align="top-center"/>
+</instance>
 </instances>
